File: PCB/DMX_usb.kicad_pcb (KiCad board)
At the start: 2 copper layers, 58.2 x 99.1 mm, 65 parts, among them IC1 FE1.1S, J1 Conn_01x02_Male, J2 Conn_01x02_Male, J3 XLR3, J4 XLR3, J5 XLR3, J6 XLR3, J7 Conn_01x02_Male, J8 Conn_01x02_Male, P1 USB_C_Plug_USB2.0, P2 USB_C_Plug_USB2.0, P3 USB_C_Plug_USB2.0, P4 USB_C_Plug_USB2.0, U1 FT232RL, U2 75176B, U3 FT232RL, U4 FT232RL, U5 FT232RL, U6 75176B, U7 75176B, U8 75176B, Y1 Crystal

Commit message: v2
fixed some stupid problems with pcb desgn
Parts:
- removed J1, J2, J7, J8: Conn_01x02_Male, Connector_PinSocket_2.54mm:PinSocket_1x02_P2.54mm_Vertical
- removed JP1: Jumper, Connector_PinSocket_2.54mm:PinSocket_1x02_P2.54mm_Vertical
- removed JP2, JP3: SolderJumper_2_Open, Jumper:SolderJumper-2_P1.3mm_Open_TrianglePad1.0x1.5mm
- removed P1, P2, P3, P4: USB_C_Plug_USB2.0, Connector_USB:USB_C_Receptacle_Palconn_UTC16-G
- added D1: LED, LED_SMD:LED_0805_2012Metric_Pad1.15x1.40mm_HandSolder, F.Cu at (221.2, 46.0)
- added D2: LED, LED_SMD:LED_0805_2012Metric_Pad1.15x1.40mm_HandSolder, F.Cu at (221.2, 48.5)
- added D3: LED, LED_SMD:LED_0805_2012Metric_Pad1.15x1.40mm_HandSolder, F.Cu at (221.5, 99.6)
- added D4: LED, LED_SMD:LED_0805_2012Metric_Pad1.15x1.40mm_HandSolder, F.Cu at (221.5, 97.0)
- added D5: LED, LED_SMD:LED_0805_2012Metric_Pad1.15x1.40mm_HandSolder, F.Cu at (221.5, 74.1)
- added D6: LED, LED_SMD:LED_0805_2012Metric_Pad1.15x1.40mm_HandSolder, F.Cu at (221.5, 71.4)
- added D7: LED, LED_SMD:LED_0805_2012Metric_Pad1.15x1.40mm_HandSolder, F.Cu at (221.2, 121.9)
- added D8: LED, LED_SMD:LED_0805_2012Metric_Pad1.15x1.40mm_HandSolder, F.Cu at (221.2, 124.5)
- added J10: DMX, Connector_PinSocket_2.54mm:PinSocket_1x03_P2.54mm_Vertical, F.Cu at (268.2, 76.1)
- added J11: DMX, Connector_PinSocket_2.54mm:PinSocket_1x03_P2.54mm_Vertical, F.Cu at (268.2, 101.3)
- added J12: DMX, Connector_PinSocket_2.54mm:PinSocket_1x03_P2.54mm_Vertical, F.Cu at (268.2, 126.5)
- added J13: USB_C, Connector_USB:USB_C_Receptacle_Palconn_UTC16-G, F.Cu at (222.2, 56.1)
- added J14: USB_C, Connector_USB:USB_C_Receptacle_Palconn_UTC16-G, F.Cu at (222.2, 81.3)
- added J15: USB_C, Connector_USB:USB_C_Receptacle_Palconn_UTC16-G, F.Cu at (222.2, 106.4)
- added J16: USB_C, Connector_USB:USB_C_Receptacle_Palconn_UTC16-G, F.Cu at (222.2, 131.6)
- added J17: USB, Connector_PinSocket_2.54mm:PinSocket_1x04_P2.54mm_Vertical, F.Cu at (242.6, 65.5)
- added J9: DMX, Connector_PinSocket_2.54mm:PinSocket_1x03_P2.54mm_Vertical, F.Cu at (268.2, 51.2)
- added R18: R, Resistor_SMD:R_0805_2012Metric_Pad1.15x1.40mm_HandSolder, F.Cu at (225.3, 74.2)
- added R19: R, Resistor_SMD:R_0805_2012Metric_Pad1.15x1.40mm_HandSolder, F.Cu at (225.3, 71.4)
- added R2: R, Resistor_SMD:R_0805_2012Metric_Pad1.15x1.40mm_HandSolder, F.Cu at (225.0, 46.0)
- added R20: R, Resistor_SMD:R_0805_2012Metric_Pad1.15x1.40mm_HandSolder, F.Cu at (225.1, 121.8)
- added R21: R, Resistor_SMD:R_0805_2012Metric_Pad1.15x1.40mm_HandSolder, F.Cu at (225.0, 124.5)
- added R6: R, Resistor_SMD:R_0805_2012Metric_Pad1.15x1.40mm_HandSolder, F.Cu at (225.1, 48.5)
- added R7: R, Resistor_SMD:R_0805_2012Metric_Pad1.15x1.40mm_HandSolder, F.Cu at (225.6, 99.6)
- added R8: R, Resistor_SMD:R_0805_2012Metric_Pad1.15x1.40mm_HandSolder, F.Cu at (225.6, 97.1)
- moved C13 5.60 mm to (249.7, 45.7), turned to 180 degrees
- moved C3 4.59 mm to (242.6, 122.7), turned to 180 degrees
- moved C6 4.58 mm to (247.9, 122.7), turned to 180 degrees
- moved C15 4.55 mm to (247.9, 98.3), turned to 180 degrees
- moved C9 4.06 mm to (243.1, 98.3), turned to 180 degrees
- moved C8 3.83 mm to (242.8, 72.9)
- moved C14 3.82 mm to (246.6, 72.9), turned to 180 degrees
- moved C7 3.06 mm to (245.1, 45.7), turned to 180 degrees
Connections:
- C1 pad 1: Net-(C1-Pad1) -> +5V
- IC1 pad 20: Net-(C1-Pad1) -> +5V
- U1 pad 17: Net-(U1-Pad17) -> Net-(C6-Pad1)
- U1 pad 26: Net-(C6-Pad1) -> GND
- U3 pad 17: Net-(U3-Pad17) -> Net-(C13-Pad1)
- U3 pad 26: Net-(C13-Pad1) -> GND
- U4 pad 17: Net-(U4-Pad17) -> Net-(C14-Pad1)
- U4 pad 26: Net-(C14-Pad1) -> GND
- U5 pad 17: Net-(U5-Pad17) -> Net-(C15-Pad1)
- U5 pad 26: Net-(C15-Pad1) -> GND
Routing:
- net +5V: track 384.1 -> 421.0 mm, vias 6 -> 9
- net Net-(R6-Pad1): track 0.00 -> 29.0 mm
- net Net-(R19-Pad1): track 0.00 -> 28.4 mm, vias 0 -> 2
- net Net-(C1-Pad1): track 28.2 -> 0.00 mm, vias 2 -> 0
- net Net-(R7-Pad1): track 0.00 -> 27.0 mm, vias 0 -> 2
- net Net-(R18-Pad1): track 0.00 -> 26.8 mm, vias 0 -> 2
- net Net-(R2-Pad1): track 0.00 -> 26.5 mm
- net Net-(R8-Pad1): track 0.00 -> 25.7 mm, vias 0 -> 2
- net Net-(R20-Pad1): track 0.00 -> 25.3 mm, vias 0 -> 2
- net Net-(R21-Pad1): track 0.00 -> 24.5 mm, vias 0 -> 2
- net Net-(IC1-Pad15): track 17.6 -> 37.5 mm
- net Net-(IC1-Pad16): track 19.2 -> 38.9 mm
- net GND: track 153.3 -> 139.7 mm, vias 32 -> 38
- net Net-(J12-Pad3): track 12.6 -> 22.7 mm
- net Net-(J4-Pad3): track 13.3 -> 22.6 mm
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Other:
- board size 58.2 x 99.1 mm -> 55 x 99.1 mm
