File: PCB/DMX_usb.sch (KiCad schematic (older format))
At the start: 65 parts, among them IC1 FE1.1S, J1 Conn_01x02_Male, J2 Conn_01x02_Male, J3 XLR3, J4 XLR3, J5 XLR3, J6 XLR3, J7 Conn_01x02_Male, J8 Conn_01x02_Male, P1 USB_C_Plug_USB2.0, P2 USB_C_Plug_USB2.0, P3 USB_C_Plug_USB2.0, P4 USB_C_Plug_USB2.0, U1 FT232RL, U2 75176B, U3 FT232RL, U4 FT232RL, U5 FT232RL, U6 75176B, U7 75176B, U8 75176B, Y1 Crystal

Commit message: v2
fixed some stupid problems with pcb desgn
Parts:
- removed J1, J2, J7, J8: Conn_01x02_Male, Connector_PinSocket_2.54mm:PinSocket_1x02_P2.54mm_Vertical, symbol Connector:Conn_01x02_Male
- removed JP1: Jumper, Connector_PinSocket_2.54mm:PinSocket_1x02_P2.54mm_Vertical, symbol Device:Jumper
- removed JP2, JP3: SolderJumper_2_Open, Jumper:SolderJumper-2_P1.3mm_Open_TrianglePad1.0x1.5mm, symbol Jumper:SolderJumper_2_Open
- removed P1, P2, P3, P4: USB_C_Plug_USB2.0, Connector_USB:USB_C_Receptacle_Palconn_UTC16-G, symbol Connector:USB_C_Plug_USB2.0
- added C24: 100nf, Capacitor_SMD:C_0805_2012Metric_Pad1.15x1.40mm_HandSolder, symbol Device:C
- added D1, D2, D3, D4, D5, D6, D7, D8: LED, LED_SMD:LED_0805_2012Metric_Pad1.15x1.40mm_HandSolder, symbol Device:LED
- added J10, J11, J12, J9: Conn_01x03, Connector_PinSocket_2.54mm:PinSocket_1x03_P2.54mm_Vertical, symbol Connector_Generic:Conn_01x03
- added J13, J14, J15, J16: USB_C_Receptacle_USB2.0, Connector_USB:USB_C_Receptacle_Palconn_UTC16-G, symbol Connector:USB_C_Receptacle_USB2.0
- added J17: Conn_01x04, Connector_PinSocket_2.54mm:PinSocket_1x04_P2.54mm_Vertical, symbol Connector_Generic:Conn_01x04
- added R18, R19, R2, R20, R21, R6, R7, R8: R, Resistor_SMD:R_0805_2012Metric_Pad1.15x1.40mm_HandSolder, symbol Device:R
- IC1: symbol SamacSys_Parts:FE1.1S -> DMX_usb-rescue:FE1.1S-SamacSys_Parts
- U2, U6, U7, U8: symbol Kicad_custom:75176B -> DMX_usb-rescue:75176B-Kicad_custom
- Y1: value Crystal -> Crystal 12MHZ
Connections:
- net +5V: now also C1.1, IC1.20 (VDD5), C24.1, D1.2 (A), D2.2 (A), D3.2 (A), D4.2 (A), D5.2 (A), D6.2 (A), D7.2 (A), D8.2 (A), J13.A4 (VBUS), J13.A9 (VBUS), J13.B4 (VBUS), J13.B9 (VBUS), J14.A4 (VBUS), J14.A9 (VBUS), J14.B4 (VBUS), J14.B9 (VBUS), J15.A4 (VBUS), J15.A9 (VBUS), J15.B4 (VBUS), J15.B9 (VBUS), J16.A4 (VBUS), J16.A9 (VBUS), J16.B4 (VBUS), J16.B9 (VBUS), J17.4 (Pin_4)
- net D2+: now also J14.A6 (D+), J14.B6 (D+)
- net D2-: now also J14.A7 (D-), J14.B7 (D-)
- net D3+: now also J15.A6 (D+), J15.B6 (D+)
- net D3-: now also J15.A7 (D-), J15.B7 (D-)
- net D4+: now also J16.A6 (D+), J16.B6 (D+)
- net D4-: now also J16.A7 (D-), J16.B7 (D-)
- net GND: now also U1.26 (TEST), U3.26 (TEST), U4.26 (TEST), U5.26 (TEST), C24.2, J13.A1 (GND), J13.A12 (GND), J13.B1 (GND), J13.B12 (GND), J13.S1 (SHIELD), J14.A1 (GND), J14.A12 (GND), J14.B1 (GND), J14.B12 (GND), J14.S1 (SHIELD), J15.A1 (GND), J15.A12 (GND), J15.B1 (GND), J15.B12 (GND), J15.S1 (SHIELD), J16.A1 (GND), J16.A12 (GND), J16.B1 (GND), J16.B12 (GND), J16.S1 (SHIELD), J17.1 (Pin_1)
- net at U3.17 (3V3OUT): now also C13.1
- net at U3.22 (CBUS1): now also R6.1
- net at U3.23 (CBUS0): now also R2.1
- net at F2.1, J4.1: now also J9.1 (Pin_1)
- net at J4.2, R10.1, R9.2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: now also J9.2 (Pin_2)
- net at J4.3, R10.2, R11.1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: now also J9.3 (Pin_3)
- net at IC1.15 (DMU): now also J13.A7 (D-), J13.B7 (D-), J17.3 (Pin_3)
- net at IC1.16 (DPU): now also J13.A6 (D+), J13.B6 (D+), J17.2 (Pin_2)
- net at U4.17 (3V3OUT): now also C14.1
- net at U4.22 (CBUS1): now also R19.1
- net at U4.23 (CBUS0): now also R18.1
- net at F3.1, J5.1: now also J10.1 (Pin_1)
- net at J5.2, R12.2, R13.1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: now also J10.2 (Pin_2)
- net at J5.3, R13.2, R14.1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: now also J10.3 (Pin_3)
- net at U5.17 (3V3OUT): now also C15.1
- net at U5.22 (CBUS1): now also R8.1
- net at U5.23 (CBUS0): now also R7.1
- net at F4.1, J6.1: now also J11.1 (Pin_1)
- net at J6.2, R15.2, R16.1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: now also J11.2 (Pin_2)
- net at J6.3, R16.2, R17.1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: now also J11.3 (Pin_3)
- net at U1.17 (3V3OUT): now also C6.1
- net at U1.22 (CBUS1): now also R21.1
- net at U1.23 (CBUS0): now also R20.1
- net at F1.1, J3.1: now also J12.1 (Pin_1)
- net at J3.2, R3.2, R4.1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: now also J12.2 (Pin_2)
- net at J3.3, R4.2, R5.1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: now also J12.3 (Pin_3)
- new net: D6.1 (K), R19.2
- new net: D5.1 (K), R18.2
- new net: D2.1 (K), R6.2
- new net: D1.1 (K), R2.2
- new net: D4.1 (K), R8.2
- new net: D3.1 (K), R7.2
- new net: D8.1 (K), R21.2
- new net: D7.1 (K), R20.2
Other:
- moved on the sheet: C13, C14, C15, C6
